File: kicad/w010lo-backplane/w010lo-backplane.kicad_pcb (KiCad board)
At the start: 4 copper layers, 99.8 x 99.8 mm, 23 parts, among them J1 Barrel_Jack, J2 VME, J3 VME, J4 VME, J5 VME, J6 VME, SW2 SW_SPST

Commit message: Final Kicad update before manufacturing
Parts:
- moved C4 4.19 mm to (107.3, 137.6), turned to 90 degrees
- moved J2 3.34 mm to (113.2, 58.8)
- moved J6 2.80 mm to (181.2, 58.9)
- moved C5 2.67 mm to (124.3, 137.7)
- moved C8 2.03 mm to (175.3, 137.7)
- moved J3 1.80 mm to (130.2, 58.9)
- moved J5 1.26 mm to (164.2, 58.9)
- moved C6 0.89 mm to (141.4, 137.7)
- moved D2 0.51 mm to (192.4, 88.3)
- moved C7 0.39 mm to (158.1, 137.7)
- moved J4 0.27 mm to (147.2, 58.9)
Connections:
- J2 pad b1: unconnected-(J2B-Pin_b1-Padb1) -> USER0
- J2 pad b10: unconnected-(J2B-Pin_b10-Padb10) -> USER9
- J2 pad b11: unconnected-(J2B-Pin_b11-Padb11) -> USER10
- J2 pad b12: unconnected-(J2B-Pin_b12-Padb12) -> USER11
- J2 pad b13: unconnected-(J2B-Pin_b13-Padb13) -> USER12
- J2 pad b14: unconnected-(J2B-Pin_b14-Padb14) -> USER13
- J2 pad b15: unconnected-(J2B-Pin_b15-Padb15) -> USER14
- J2 pad b2: unconnected-(J2B-Pin_b2-Padb2) -> USER1
- J2 pad b21: unconnected-(J2B-Pin_b21-Padb21) -> USER15
- J2 pad b22: unconnected-(J2B-Pin_b22-Padb22) -> USER16
- J2 pad b3: unconnected-(J2B-Pin_b3-Padb3) -> USER2
- J2 pad b4: unconnected-(J2B-Pin_b4-Padb4) -> USER3
- J2 pad b5: unconnected-(J2B-Pin_b5-Padb5) -> USER4
- J2 pad b6: unconnected-(J2B-Pin_b6-Padb6) -> USER5
- J2 pad b7: unconnected-(J2B-Pin_b7-Padb7) -> USER6
- J2 pad b8: unconnected-(J2B-Pin_b8-Padb8) -> USER7
- J2 pad b9: unconnected-(J2B-Pin_b9-Padb9) -> USER8
- J2 pad c10: unconnected-(J2C-Pin_c10-Padc10) -> ~{IO}
- J3 pad b1: unconnected-(J3B-Pin_b1-Padb1) -> USER0
- J3 pad b10: unconnected-(J3B-Pin_b10-Padb10) -> USER9
- J3 pad b11: unconnected-(J3B-Pin_b11-Padb11) -> USER10
- J3 pad b12: unconnected-(J3B-Pin_b12-Padb12) -> USER11
- J3 pad b13: unconnected-(J3B-Pin_b13-Padb13) -> USER12
- J3 pad b14: unconnected-(J3B-Pin_b14-Padb14) -> USER13
- J3 pad b15: unconnected-(J3B-Pin_b15-Padb15) -> USER14
- J3 pad b2: unconnected-(J3B-Pin_b2-Padb2) -> USER1
- J3 pad b21: unconnected-(J3B-Pin_b21-Padb21) -> USER15
- J3 pad b22: unconnected-(J3B-Pin_b22-Padb22) -> USER16
- J3 pad b3: unconnected-(J3B-Pin_b3-Padb3) -> USER2
- J3 pad b4: unconnected-(J3B-Pin_b4-Padb4) -> USER3
- J3 pad b5: unconnected-(J3B-Pin_b5-Padb5) -> USER4
- J3 pad b6: unconnected-(J3B-Pin_b6-Padb6) -> USER5
- J3 pad b7: unconnected-(J3B-Pin_b7-Padb7) -> USER6
- J3 pad b8: unconnected-(J3B-Pin_b8-Padb8) -> USER7
- J3 pad b9: unconnected-(J3B-Pin_b9-Padb9) -> USER8
- J3 pad c10: unconnected-(J3C-Pin_c10-Padc10) -> ~{IO}
- J4 pad b1: unconnected-(J4B-Pin_b1-Padb1) -> USER0
- J4 pad b10: unconnected-(J4B-Pin_b10-Padb10) -> USER9
- J4 pad b11: unconnected-(J4B-Pin_b11-Padb11) -> USER10
- J4 pad b12: unconnected-(J4B-Pin_b12-Padb12) -> USER11
- J4 pad b13: unconnected-(J4B-Pin_b13-Padb13) -> USER12
- J4 pad b14: unconnected-(J4B-Pin_b14-Padb14) -> USER13
- J4 pad b15: unconnected-(J4B-Pin_b15-Padb15) -> USER14
- J4 pad b2: unconnected-(J4B-Pin_b2-Padb2) -> USER1
- J4 pad b21: unconnected-(J4B-Pin_b21-Padb21) -> USER15
- J4 pad b22: unconnected-(J4B-Pin_b22-Padb22) -> USER16
- J4 pad b3: unconnected-(J4B-Pin_b3-Padb3) -> USER2
- J4 pad b4: unconnected-(J4B-Pin_b4-Padb4) -> USER3
- J4 pad b5: unconnected-(J4B-Pin_b5-Padb5) -> USER4
- J4 pad b6: unconnected-(J4B-Pin_b6-Padb6) -> USER5
- J4 pad b7: unconnected-(J4B-Pin_b7-Padb7) -> USER6
- J4 pad b8: unconnected-(J4B-Pin_b8-Padb8) -> USER7
- J4 pad b9: unconnected-(J4B-Pin_b9-Padb9) -> USER8
- J4 pad c10: unconnected-(J4C-Pin_c10-Padc10) -> ~{IO}
- J5 pad b1: unconnected-(J5B-Pin_b1-Padb1) -> USER0
- J5 pad b10: unconnected-(J5B-Pin_b10-Padb10) -> USER9
- J5 pad b11: unconnected-(J5B-Pin_b11-Padb11) -> USER10
- J5 pad b12: unconnected-(J5B-Pin_b12-Padb12) -> USER11
- J5 pad b13: unconnected-(J5B-Pin_b13-Padb13) -> USER12
- J5 pad b14: unconnected-(J5B-Pin_b14-Padb14) -> USER13
- J5 pad b15: unconnected-(J5B-Pin_b15-Padb15) -> USER14
- J5 pad b2: unconnected-(J5B-Pin_b2-Padb2) -> USER1
- J5 pad b21: unconnected-(J5B-Pin_b21-Padb21) -> USER15
- J5 pad b22: unconnected-(J5B-Pin_b22-Padb22) -> USER16
- J5 pad b3: unconnected-(J5B-Pin_b3-Padb3) -> USER2
- J5 pad b4: unconnected-(J5B-Pin_b4-Padb4) -> USER3
- J5 pad b5: unconnected-(J5B-Pin_b5-Padb5) -> USER4
- J5 pad b6: unconnected-(J5B-Pin_b6-Padb6) -> USER5
- J5 pad b7: unconnected-(J5B-Pin_b7-Padb7) -> USER6
- J5 pad b8: unconnected-(J5B-Pin_b8-Padb8) -> USER7
- J5 pad b9: unconnected-(J5B-Pin_b9-Padb9) -> USER8
- J5 pad c10: unconnected-(J5C-Pin_c10-Padc10) -> ~{IO}
- J6 pad a22: ~{IACKOUT5} -> unconnected-(J6A-Pin_a22-Pada22)
- J6 pad b1: unconnected-(J6B-Pin_b1-Padb1) -> USER0
- J6 pad b10: unconnected-(J6B-Pin_b10-Padb10) -> USER9
- J6 pad b11: unconnected-(J6B-Pin_b11-Padb11) -> USER10
- J6 pad b12: unconnected-(J6B-Pin_b12-Padb12) -> USER11
- J6 pad b13: unconnected-(J6B-Pin_b13-Padb13) -> USER12
- J6 pad b14: unconnected-(J6B-Pin_b14-Padb14) -> USER13
- J6 pad b15: unconnected-(J6B-Pin_b15-Padb15) -> USER14
- J6 pad b2: unconnected-(J6B-Pin_b2-Padb2) -> USER1
- J6 pad b21: unconnected-(J6B-Pin_b21-Padb21) -> USER15
- J6 pad b22: unconnected-(J6B-Pin_b22-Padb22) -> USER16
- J6 pad b3: unconnected-(J6B-Pin_b3-Padb3) -> USER2
- J6 pad b4: unconnected-(J6B-Pin_b4-Padb4) -> USER3
- J6 pad b5: unconnected-(J6B-Pin_b5-Padb5) -> USER4
- J6 pad b6: unconnected-(J6B-Pin_b6-Padb6) -> USER5
- J6 pad b7: unconnected-(J6B-Pin_b7-Padb7) -> USER6
- J6 pad b8: unconnected-(J6B-Pin_b8-Padb8) -> USER7
- J6 pad b9: unconnected-(J6B-Pin_b9-Padb9) -> USER8
- J6 pad c10: unconnected-(J6C-Pin_c10-Padc10) -> ~{IO}
Routing:
- net USER9: track 0.00 -> 72.3 mm
- net USER2: track 0.00 -> 72.3 mm
- net USER7: track 0.00 -> 72.3 mm
- net USER1: track 0.00 -> 72.3 mm
- net USER16: track 0.00 -> 72.3 mm
- net USER6: track 0.00 -> 72.1 mm
- net USER5: track 0.00 -> 72.1 mm
- net USER4: track 0.00 -> 71.9 mm
- net USER12: track 0.00 -> 71.9 mm
- net USER3: track 0.00 -> 71.9 mm
- net USER11: track 0.00 -> 71.9 mm
- net ~{IO}: track 0.00 -> 71.5 mm
- net USER0: track 0.00 -> 71.5 mm
- net USER13: track 0.00 -> 71.5 mm
- net USER15: track 0.00 -> 71.4 mm
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Other:
- board text added: "DC 9V IN"
- board text added: "POWER"
- board text added: "SLOT 1"
- board text added: "SLOT 2"
- board text added: "SLOT 3"
- board text added: "SLOT 4"
- board text added: "SLOT 5"
- board text added: "w010lo backplane rev. 0.4 07/28/2026"
- board text removed: "w010lo backplane rev. 0.2 07/12/2026"
