File: kicad/w010lo-backplane/w010lo-backplane.kicad_sch (KiCad schematic)
At the start: 15 parts, among them J1 Barrel_Jack, J2 VME, SW2 SW_SPST

Commit message: Final Kicad update before manufacturing
Connections:
- net ~{IO}: now reaches J2.c10 (Pin_c10)
- net USER0: now reaches J2.b1 (Pin_b1)
- net USER9: now reaches J2.b10 (Pin_b10)
- net USER10: now reaches J2.b11 (Pin_b11)
- net USER11: now reaches J2.b12 (Pin_b12)
- net USER12: now reaches J2.b13 (Pin_b13)
- net USER13: now reaches J2.b14 (Pin_b14)
- net USER14: now reaches J2.b15 (Pin_b15)
- net USER1: now reaches J2.b2 (Pin_b2)
- net USER15: now reaches J2.b21 (Pin_b21)
- net USER16: now reaches J2.b22 (Pin_b22)
- net USER2: now reaches J2.b3 (Pin_b3)
- net USER3: now reaches J2.b4 (Pin_b4)
- net USER4: now reaches J2.b5 (Pin_b5)
- net USER5: now reaches J2.b6 (Pin_b6)
- net USER6: now reaches J2.b7 (Pin_b7)
- net USER7: now reaches J2.b8 (Pin_b8)
- net USER8: now reaches J2.b9 (Pin_b9)
- no-connect marks 23 -> 3
