File: kicad/w010lo-io/w010lo-io.kicad_sch (KiCad schematic)
At the start: 14 parts, among them J1 DE9_Pins, J2 VME, J3 Conn_01x06, U1 68681, U3 MAX232, Y1 3.6864 MHz

Commit message: Final Kicad update before manufacturing
Parts:
- added C6: 0.1uF, Capacitor_THT:C_Disc_D5.0mm_W2.5mm_P5.00mm, symbol Device:C
- added D1, D2, D3: SD103, Diode_THT:D_DO-35_SOD27_P7.62mm_Horizontal, symbol Device:D_Schottky
- added R3: 4.7k, Resistor_THT:R_Axial_DIN0207_L6.3mm_D2.5mm_P7.62mm_Horizontal, symbol Device:R
- C1: footprint (none) -> Capacitor_THT:C_Disc_D5.0mm_W2.5mm_P5.00mm
- C2, C3, C4, C5: footprint (none) -> Capacitor_THT:CP_Radial_D5.0mm_P2.50mm
- J1: footprint (none) -> custom:DE-9-Amphenol
- J3: footprint (none) -> Connector_PinHeader_2.54mm:PinHeader_1x06_P2.54mm_Horizontal
- U1: footprint (none) -> Package_DIP:DIP-40_W15.24mm_Socket
- U2: footprint (none) -> Package_DIP:DIP-24_W7.62mm_Socket
- U3: footprint (none) -> Package_DIP:DIP-16_W7.62mm_Socket
Connections:
- net A1: now also U2.3 (IN)
- net A12: now also U2.1 (CLK/IN)
- net A13: now also U2.2 (IN)
- net A2: now also U2.4 (IN/PD)
- net A3: now also U2.5 (IN)
- net GND: now also C6.2
- net R/~{W}: now also U2.8 (IN)
- net VCC: now also C6.1, R3.1
- net ~{AS}: now also U2.7 (IN)
- net ~{DTACK}: now also D1.2 (A)
- net ~{DUARTCS}: now also U2.22 (I/O); no longer U2.23 (I/O)
- net ~{IACKIN}: now also U2.6 (IN); no longer U1.37 (IACK)
- net ~{IACKOUT}: now also U2.23 (I/O)
- net ~{LDS}: now also U2.9 (IN)
- net ~{UDS}: now also U2.10 (IN)
- net ~{VPA}: now also U2.17 (I/O)
- net ~{IO}: now reaches U2.11 (IN)
- net ~{IO}: now also J2.c10 (Pin_c10)
- net ~{ATAWR}: now reaches U2.14 (I/O)
- net ~{ATAWR}: now also D3.1 (K)
- net ~{ATARD}: now reaches U2.15 (I/O)
- net ~{ATARD}: now also D2.1 (K)
- net at U2.16 (I/O): now also D1.1 (K)
- net ~{WR}: now reaches U2.18 (I/O)
- net ~{RD}: now reaches U2.19 (I/O)
- net ~{RTCCS}: now reaches U2.20 (I/O)
- net ~{DUARTIACK}: now reaches U2.21 (I/O)
- net ~{DUARTIACK}: now also U1.37 (IACK)
- new net ~{BUFOE}: D2.2 (A), D3.2 (A), R3.2
Other:
- added sheet PATA (pata.kicad_sch)
- added sheet RTC (rtc.kicad_sch)
