File: kicad/w010lo-cpu/w010lo-cpu.kicad_pcb (KiCad board)
At the start: 4 copper layers, 99.8 x 99.8 mm, 23 parts, among them J2 VME, SW1 SW_Push, U1 MC68010P, U2 74LS05, U3 74LS175, U4 74LS148, U5 TC1232, U6 GAL16V8, Y1 12MHz

Commit message: Final Kicad update before manufacturing
Parts:
- moved SW1 42.6 mm to (153.8, 139.9), turned to 0 degrees
Routing:
- net Net-(U5-~{PB}): track 62.8 -> 52.2 mm
Other:
- board text added: "74HCT05"
- board text added: "74HCT175"
- board text added: "74LS148"
- board text added: "GAL"
- board text added: "MC68010"
- board text added: "RESET"
- board text added: "TC1232"
- board text added: "w010lo CPU Board r0.2 07/26/2026"
- board text removed: "w010lo CPU Board r0.1 07/19/2026"

Commit message: Add fixes to kicad + new addrs in demos
Parts:
- removed R3: 4.7k, Resistor_THT:R_Axial_DIN0204_L3.6mm_D1.6mm_P5.08mm_Horizontal
Connections:
- RN2 pad 2: unconnected-(RN2-R1-Pad2) -> ~{BERR}
- U4 pad 5: Net-(U4-EI) -> GND
Routing:
- net ~{BERR}: track 100.4 -> 139.4 mm, vias 1 -> 2
- net Net-(U4-EI): track 12.8 -> 0.00 mm
- net A1: track 39.3 -> 40.3 mm
Other:
- board text added: "w010lo CPU Board r1 08/09/2026"
- board text removed: "w010lo CPU Board r0.2 07/26/2026"
Changed lines of the file:
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@@
 		)
 	)
-	(footprint "Resistor_THT:R_Axial_DIN0204_L3.6mm_D1.6mm_P5.08mm_Horizontal"
-		(layer "F.Cu")
-		(at 149.86 85.09 90)
-		(descr "Resistor, Axial_DIN0204 series, Axial, Horizontal, pin pitch=5.08mm, 0.167W, length*diameter=3.6*1.6mm^2, http://cdn-reichelt.de/documents/datenblatt/B400/1_4W%23YAG.pdf")
-		(tags "Resistor Axial_DIN0204 series Axial Horizontal pin pitch 5.08mm 0.167W length 3.6mm diameter 1.6mm")
-		(property "Reference" "R3"
-			(at 6.858 0 180)
-			(layer "F.SilkS")
-			(effects
-				(font
-					(size 1 1)
-					(thickness 0.15)
-				)
-			)
-		)
-		(property "Value" "4.7k"
-			(at 2.54 1.92 90)
-			(layer "F.Fab")
-			(effects
-				(font
-					(size 1 1)
-					(thickness 0.15)
-				)
-			)
-		)
-		(property "Datasheet" ""
-			(at 0 0 90)
-			(layer "F.Fab")
-			(hide yes)
-			(effects
-				(font
-					(size 1.27 1.27)
-				)
-			)
-		)
-		(property "Description" "Resistor"
-			(at 0 0 90)
-			(layer "F.Fab")
-			(hide yes)
-			(effects
-				(font
-					(size 1.27 1.27)
-				)
-			)
-		)
-		(property "KiLib_Generator" "resistor/THT"
-			(at 0 0 90)
-			(layer "F.SilkS")
-			(hide yes)
-			(effects
-				(font
-					(size 1 1)
-					(thickness 0.15)
-				)
-			)
-		)
-		(property ki_fp_filters "R_*")
-		(sheetname "/")
-		(sheetfile "w010lo-cpu.kicad_sch")
-		(units
-			(unit
-				(name "A")
-				(pins "1" "2")
-			)
-		)
-		(attr through_hole)
-		(duplicate_pad_numbers_are_jumpers no)
-		(fp_line
-			(start 0.62 -0.92)
-			(end 4.46 -0.92)
-			(stroke
-				(width 0.12)
-				(type solid)
-			)
-			(layer "F.SilkS")
-		)
-		(fp_line
-			(start 0.62 0.92)
-			(end 4.46 0.92)
-			(stroke
-				(width 0.12)
-				(type solid)
-			)
-			(layer "F.SilkS")
-		)
-		(fp_rect
-			(start -0.95 -1.05)
-			(end 6.03 1.05)
-			(stroke
-				(width 0.05)
-				(type solid)
-			)
-			(fill no)
-			(layer "F.CrtYd")
-		)
-		(fp_line
-			(start 5.08 0)
-			(end 4.34 0)
-			(stroke
-				(width 0.1)
-				(type solid)
-			)
-			(layer "F.Fab")
-		)
-		(fp_line
-			(start 0 0)
-			(end 0.74 0)
-			(stroke
-				(width 0.1)
-				(type solid)
-			)
-			(layer "F.Fab")
-		)
-		(fp_rect
-			(start 0.74 -0.8)
-			(end 4.34 0.8)
-			(stroke
-				(width 0.1)
-				(type solid)
-			)
-			(fill no)
-			(layer "F.Fab")
-		)
-		(fp_text user "${REFERENCE}"
-			(at 2.54 0 90)
-			(layer "F.Fab")
-			(effects
-				(font
-					(size 0.72 0.72)
-					(thickness 0.108)
-				)
-			)
-		)
-		(pad "1" thru_hole circle
-			(at 0 0 90)
-			(size 1.4 1.4)
-			(drill 0.7)
-			(layers "*.Cu" "*.Mask")
-			(remove_unused_layers no)
-			(net "VCC")
-			(pintype "passive")
-		)
-		(pad "2" thru_hole circle
-			(at 5.08 0 90)
-			(size 1.4 1.4)
-			(drill 0.7)
-			(layers "*.Cu" "*.Mask")
-			(remove_unused_layers no)
-			(net "Net-(U4-EI)")
-			(pintype "passive")
-		)
-		(embedded_fonts no)
-		(model "${KICAD10_3DMODEL_DIR}/Resistor_THT.3dshapes/R_Axial_DIN0204_L3.6mm_D1.6mm_P5.08mm_Horizontal.step"
-			(offset
-				(xyz 0 0 0)
-			)
-			(scale
-				(xyz 1 1 1)
-			)
-			(rotate
-				(xyz 0 0 0)
-			)
-		)
-	)
 	(footprint "MountingHole:MountingHole_3.2mm_M3"
 		(layer "F.Cu")
@@
 			(layers "*.Cu" "*.Mask")
 			(remove_unused_layers no)
-			(net "Net-(U4-EI)")
+			(net "GND")
 			(pinfunction "EI_5")
 			(pintype "input")
@@
 			(layers "*.Cu" "*.Mask")
 			(remove_unused_layers no)
-			(net "unconnected-(RN2-R1-Pad2)")
+			(net "~{BERR}")
 			(pinfunction "R1_2")
-			(pintype "passive+no_connect")
+			(pintype "passive")
 		)
 		(pad "3" thru_hole circle
@@
 		(layer "Edge.Cuts")
 	)
-	(gr_text "w010lo CPU Board\nr0.2 07/26/2026"
+	(gr_text "w010lo CPU Board\nr1 08/09/2026"
 		(at 130.81 141.986 0)
 		(layer "F.SilkS")
@@
 	)
 	(segment
-		(start 143.986365 79.248)
-		(end 145.426365 80.688)
-		(width 0.1524)
-		(layer "B.Cu")
-		(net "Net-(U4-EI)")
-	)
-	(segment
-		(start 149.182 80.688)
-		(end 149.86 80.01)
-		(width 0.1524)
-		(layer "B.Cu")
-		(net "Net-(U4-EI)")
-	)
-	(segment
-		(start 145.426365 80.688)
-		(end 149.182 80.688)
-		(width 0.1524)
-		(layer "B.Cu")
-		(net "Net-(U4-EI)")
-	)
-	(segment
-		(start 137.922 79.248)
-		(end 143.986365 79.248)
-		(width 0.1524)
-		(layer "B.Cu")
-		(net "Net-(U4-EI)")
-	)
-	(segment
 		(start 152.124223 100.0158)
 		(end 152.628177 100.0158)
@@
 	)
 	(segment
+		(start 114.173 62.992)
+		(end 113.919 62.738)
+		(width 0.1524)
+		(layer "F.Cu")
+		(net "~{BERR}")
+	)
+	(segment
 		(start 126.233 82.034977)
 		(end 132.529823 88.3318)
@@
 	)
 	(segment
+		(start 113.919 62.738)
+		(end 99.06 62.738)
+		(width 0.1524)
+		(layer "F.Cu")
+		(net "~{BERR}")
+	)
+	(segment
 		(start 132.529823 88.3318)
 		(end 139.3858 88.3318)
@@
 		(net "~{BERR}")
 	)
+	(via
+		(at 114.173 62.992)
+		(size 0.6)
+		(drill 0.3)
+		(layers "F.Cu" "B.Cu")
+		(net "~{BERR}")
+	)
 	(segment
 		(start 126.233 81.788)
@@
 	)
 	(segment
+		(start 126.233 81.788)
+		(end 114.173 69.728)
+		(width 0.1524)
+		(layer "B.Cu")
+		(net "~{BERR}")
+	)
+	(segment
 		(start 149.980714 113.7318)
 		(end 154.3718 113.7318)
@@
 	)
 	(segment
+		(start 114.173 69.728)
+		(end 114.173 62.992)
+		(width 0.1524)
+		(layer "B.Cu")
+		(net "~{BERR}")
+	)
+	(segment
 		(start 146.304 92.964)
 		(end 146.304 110.055086)
@@
 	)
 	(segment
-		(start 125.133 62.908)
-		(end 126.233 64.008)
+		(start 90.551 59.944)
+		(end 96.774 59.944)
 		(width 0.2)
 		(layer "F.Cu")
@@
 	)
 	(segment
-		(start 98.298 61.468)
-		(end 101.817365 61.468)
+		(start 101.817365 61.468)
+		(end 102.960365 60.325)
 		(width 0.2)
 		(layer "F.Cu")
@@
 	)
 	(segment
-		(start 103.257365 62.908)
-		(end 125.133 62.908)
+		(start 89.154 61.341)
+		(end 90.551 59.944)
 		(width 0.2)
 		(layer "F.Cu")
@@
 	)
 	(segment
-		(start 101.817365 61.468)
-		(end 103.257365 62.908)
+		(start 98.298 61.468)
+		(end 101.817365 61.468)
 		(width 0.2)
 		(layer "F.Cu")
@@
 	)
 	(segment
-		(start 89.154 61.341)
-		(end 90.551 59.944)
+		(start 122.55 60.325)
+		(end 126.233 64.008)
 		(width 0.2)
 		(layer "F.Cu")
@@
 	)
 	(segment
-		(start 90.551 59.944)
-		(end 96.774 59.944)
+		(start 96.774 59.944)
+		(end 98.298 61.468)
 		(width 0.2)
 		(layer "F.Cu")
@@
 	)
 	(segment
-		(start 96.774 59.944)
-		(end 98.298 61.468)
+		(start 102.960365 60.325)
+		(end 122.55 60.325)
 		(width 0.2)
 		(layer "F.Cu")
