File: kicad/w010lo-mem/w010lo-mem.kicad_pcb (KiCad board)
At the start: 4 copper layers, 99.8 x 99.8 mm, 17 parts, among them J2 VME

Commit message: Final Kicad update before manufacturing
Parts:
- U1: renamed from UPPER ROM
- U2: renamed from LOWER ROM
- U5: renamed from UPPER RAM
- U6: renamed from LOWER RAM
- moved D1 7.56 mm to (169.9, 110.7), turned to -90 degrees
- moved C2 6.42 mm to (176.8, 67.5), turned to 90 degrees
- moved C5 4.30 mm to (110.2, 79.8)
- moved C6 3.85 mm to (136.9, 79.8)
- moved U5 3.56 mm to (130.0, 80.0)
- moved U6 3.56 mm to (156.0, 80.0)
- moved H1 0.13 mm to (190.2, 40.0)
- moved H2 0.13 mm to (190.2, 131.7)
- renumbered GAL to U3, 74HCT164 to U4
Connections:
- D1 pad 1: ~{DTACK} -> Net-(D1-K)
- D1 pad 2: Net-(D1-A) -> ~{DTACK}
- J2 pad c10: unconnected-(J2C-Pin_c10-Padc10) -> ~{IO}
- U1 pad 31: VCC -> ~{WR}
- U2 pad 31: VCC -> ~{WR}
- U3 pad 10: ~{WR} -> unconnected-(U3-IN-Pad10)
- U3 pad 11: ~{RD} -> ~{UDS}
- U3 pad 14: unconnected-(U3-I/O-Pad14) -> ~{RD}
- U3 pad 15: unconnected-(U3-I/O-Pad15) -> ~{WR}
- U3 pad 16: ~{UDS} -> ~{IO}
- U3 pad 19: Net-(D1-A) -> Net-(D1-K)
Routing:
- net ~{IO}: track 0.00 -> 129.7 mm
- net ~{WR}: track 73.4 -> 121.3 mm, vias 1 -> 2
- net Net-(D1-K): track 0.00 -> 30.0 mm
- net Net-(D1-A): track 30.0 -> 0.00 mm
- net ~{RD}: track 134.3 -> 142.5 mm, vias 0 -> 1
- net ~{URAMCS}: track 91.8 -> 97.0 mm, vias 2 -> 0
- net D6: track 181.1 -> 186.1 mm
- net D5: track 180.3 -> 185.1 mm
- net D10: track 108.0 -> 112.6 mm
- net D4: track 179.3 -> 183.6 mm
- net D11: track 113.0 -> 117.2 mm
- net D14: track 99.0 -> 103.0 mm
- net D15: track 94.4 -> 98.1 mm
- net D1: track 129.9 -> 133.4 mm
- net D0: track 121.4 -> 124.9 mm
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Other:
- board text added: "74HCT164"
- board text added: "GAL"
- board text added: "LOWER RAM"
- board text added: "LOWER ROM"
- board text added: "UPPER RAM"
- board text added: "UPPER ROM"
- board text added: "w010lo Memory Board r0.4 07/27/2026"
- board text removed: "w010lo Memory Board r0.1 07/10/2026"

Commit message: Add fixes to kicad + new addrs in demos
Connections:
- U4 pad 5: ~{REROM} -> unconnected-(U4-Q2-Pad5)
- U4 pad 6: unconnected-(U4-Q3-Pad6) -> ~{REROM}
Routing:
- net ~{REROM}: track 15.8 -> 13.2 mm
Other:
- board text added: "w010lo Memory Board r1 08/09/2026"
- board text removed: "w010lo Memory Board r0.4 07/27/2026"
Changed lines of the file:
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@@
 			(layers "*.Cu" "*.Mask")
 			(remove_unused_layers no)
-			(net "~{REROM}")
+			(net "unconnected-(U4-Q2-Pad5)")
 			(pinfunction "Q2_5")
-			(pintype "output")
+			(pintype "output+no_connect")
 		)
 		(pad "6" thru_hole circle
@@
 			(layers "*.Cu" "*.Mask")
 			(remove_unused_layers no)
-			(net "unconnected-(U4-Q3-Pad6)")
+			(net "~{REROM}")
 			(pinfunction "Q3_6")
-			(pintype "output+no_connect")
+			(pintype "output")
 		)
 		(pad "7" thru_hole circle
@@
 		)
 	)
-	(gr_text "w010lo Memory Board\nr0.4 07/27/2026"
+	(gr_text "w010lo Memory Board\nr1 08/09/2026"
 		(at 127.508 134.366 0)
 		(layer "F.SilkS")
@@
 	)
 	(segment
-		(start 177.884 97.701)
-		(end 176.784 98.801)
+		(start 177.884 92.372)
+		(end 177.884 97.701)
 		(width 0.2)
 		(layer "F.Cu")
@@
 	)
 	(segment
-		(start 177.884 89.832)
-		(end 177.884 97.701)
+		(start 182.372 87.884)
+		(end 177.884 92.372)
 		(width 0.2)
 		(layer "F.Cu")
@@
 	)
 	(segment
-		(start 182.372 85.344)
-		(end 177.884 89.832)
+		(start 177.884 97.701)
+		(end 176.784 98.801)
 		(width 0.2)
 		(layer "F.Cu")
