File: kicad/w010lo-mem/w010lo-mem.kicad_sch (KiCad schematic)
At the start: 17 parts, among them J2 VME, U1 SST39SF010, U2 SST39SF010, U4 74HCT164, U5 AS6C4008, U6 AS6C4008

Commit message: Final Kicad update before manufacturing
Connections:
- net VCC: no longer U1.31 (PGM), U2.31 (PGM)
- net ~{DTACK}: now also D1.2 (A); no longer D1.1 (K)
- net ~{RD}: now also U3.14 (I/O); no longer U3.11 (IN)
- net ~{UDS}: now also U3.11 (IN); no longer U3.16 (I/O)
- net ~{WR}: now also U1.31 (PGM), U2.31 (PGM), U3.15 (I/O); no longer U3.10 (IN)
- net at U3.19 (I/O): now also D1.1 (K); no longer D1.2 (A)
- net ~{IO}: now reaches J2.c10 (Pin_c10)
- net ~{IO}: now also U3.16 (I/O)
- no-connect marks 36 -> 34

Commit message: Add fixes to kicad + new addrs in demos
Connections:
- net ~{REROM}: now also U4.6 (Q3); no longer U4.5 (Q2)
Changed lines of the file:
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@@
 	)
 	(no_connect
-		(at 49.53 73.66)
-	)
-	(no_connect
 		(at 96.52 151.13)
 	)
@@
 	)
 	(no_connect
+		(at 49.53 71.12)
+	)
+	(no_connect
 		(at 60.96 173.99)
 	)
@@
 		)
 	)
-	(global_label "~{REROM}"
-		(shape output)
-		(at 49.53 71.12 0)
-		(fields_autoplaced yes)
-		(effects
-			(font
-				(size 1.27 1.27)
-			)
-			(justify left)
-		)
-		(property "Intersheetrefs" "${INTERSHEET_REFS}"
-			(at 58.9861 71.12 0)
-			(hide yes)
-			(show_name no)
-			(do_not_autoplace no)
-			(effects
-				(font
-					(size 1.27 1.27)
-				)
-				(justify left)
-			)
-		)
-	)
 	(global_label "D[0..7]"
 		(shape tri_state)
@@
 			(hide yes)
 			(show_name no)
+			(do_not_autoplace no)
+			(effects
+				(font
+					(size 1.27 1.27)
+				)
+				(justify left)
+			)
+		)
+	)
+	(global_label "~{REROM}"
+		(shape output)
+		(at 49.53 73.66 0)
+		(fields_autoplaced yes)
+		(effects
+			(font
+				(size 1.27 1.27)
+			)
+			(justify left)
+		)
+		(property "Intersheetrefs" "${INTERSHEET_REFS}"
+			(at 58.9861 73.66 0)
+			(hide yes)
+			(show_name no)
